File: USB-breaker/schematic.brd (EAGLE design)
At the start: 67.5 x 45.5 mm, 23 parts, among them K1 G6K-2P, K2 G6K-2P, T1 BC558B, T2 BC548B, X1 PN61729-S, X2 PN87520-S, X3 10104110, X4 UX60SC-MB-5ST

Commit message: Value of R1 changed from 120 Ω to 100 Ω. Otherwise the voltage for relay K1 is too low.
Parts:
- R1: value 120 -> 100
Changed lines of the file:
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@@
 </autorouter>
 <elements>
-<element name="R1" library="resistor" package="0207/10" value="120" x="34.29" y="43.18" smashed="yes" rot="R180">
+<element name="R1" library="resistor" package="0207/10" value="100" x="34.29" y="43.18" smashed="yes" rot="R180">
 <attribute name="NAME" x="31.623" y="42.291" size="1.27" layer="25" ratio="10" rot="R180"/>
 <attribute name="VALUE" x="36.5506" y="43.815" size="1.27" layer="27" ratio="10" rot="R180"/>
