File: USB-breaker/schematic.sch (EAGLE design)
At the start: 27 parts, among them K1 G6K-2P, K2 G6K-2P, T1 BC558B, T2 BC548B, X1 PN61729-S, X2 PN87520-S, X3 10104110, X4 UX60SC-MB-5ST

Commit message: Value of R1 changed from 120 Ω to 100 Ω. Otherwise the voltage for relay K1 is too low.
Parts:
- R1: value 120 -> 100
Changed lines of the file:
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@@
 <parts>
 <part name="FRAME1" library="frames" deviceset="DINA5_L" device=""/>
-<part name="R1" library="resistor" deviceset="R-EU_" device="0207/10" value="120"/>
+<part name="R1" library="resistor" deviceset="R-EU_" device="0207/10" value="100"/>
 <part name="C1" library="resistor" deviceset="CPOL-EU" device="E3.5-8" value="470µ"/>
 <part name="D1" library="diode" deviceset="1N4004" device=""/>
