File: LCR-Shoe/PCB/LCR-Shoe.kicad_pcb (KiCad board)
At the start: 2 copper layers, 65 x 65 mm, 30 parts, among them J1 USB_B, J2 USB_C_Receptacle, J3 USB_B_Mini, J4 USB_B_Micro, J5 Conn_01x01_Female, J6 Conn_01x01_Male, Q1 IRLML6402PbF, U1 LM2731YMF, U2 LTC4412xS6

Commit message: Improved component placement and routing.
- The USB mini B connector J3 sits now flush with the PCB edge.
- The USB micro B connector J4 was a bit too "over the edge".
- The routing near a mounting hole of the battery holder BT1 needed more clearance to the screw nut.
- The silkscreen right near the battery contacts had still the wrong polarity (see 9dcf1bd3df9cb531acfb7521de53179e96330a9a)
Parts:
- moved J3 0.90 mm to (114.0, 109.5)
- moved J4 0.75 mm to (134.4, 105.0)
Connections:
- J5 pad : (no net) -> GND
Routing:
- net +5V: track 79.9 -> 74.5 mm
- net GND: track 155.3 -> 156.2 mm
Other:
- board text added: "Rev. 20/2"
- board text removed: "Rev. 19/1"
