File: BreadBoard-Power-BusBar/BBPBB.kicad_pcb (KiCad board)
At the start: 4 copper layers, 53.8 x 5.2 mm, 11 parts, among them J1 Conn_02x02_Odd_Even, J2 Conn_02x02_Odd_Even, Q1 BC847B, SW1 JS102011JCQN

Commit message: Added interactive BOM.
Parts:
- D4: value Everlight 17-21SYGC -> 17-21SYGC
Changed lines of the file:
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@@
       (effects (font (size 0.8 0.8) (thickness 0.1)))
     )
-    (fp_text value "Everlight 17-21SYGC" (at 0 1.65) (layer F.Fab)
+    (fp_text value 17-21SYGC (at 0 1.65) (layer F.Fab)
       (effects (font (size 1 1) (thickness 0.15)))
     )
