File: breakout_boards/MCP73831-BB/MCP73831-BB.sch (KiCad schematic (older format))
At the start: 14 parts, among them J1 USB_B_Mini, J2 Conn_01x02, J3 Conn_01x04, U1 MCP73831

Commit message: The PCB is done, except for the Silk layer.
Connections:
- net PROG: now reaches R1.1, U1.5 (PROG)
Other:
- note added: "Charging"
- note added: "Done"
Changed lines of the file:
@@
 Wire Wire Line
 	4500 4050 4500 3900
+Text Notes 7950 4400 0    50   ~ 0
+Charging
+Text Notes 7050 4400 0    50   ~ 0
+Done
+Text Label 4850 3350 0    50   ~ 0
+PROG
 $EndSCHEMATC

Commit message: Add more characteristics info to standard parts.
Parts:
- R1: Characteristics (none) -> 1%,
- R2: Characteristics (none) -> 1%
- R3, R4: Characteristics (none) -> 1%, min. 0.1 W
- RV1: value 100 kΩ -> 3361P-1-104G; Characteristics (none) -> 150 kΩ
Other:
- note added: "150 kΩ"
- note added: "Imax: 402 mA due to R1"
- note removed: "Imax: 401 mA due to R1"
Changed lines of the file:
@@
 F 2 "Resistor_SMD:R_0805_2012Metric_Pad1.20x1.40mm_HandSolder" V 4680 3600 50  0001 C CNN
 F 3 "~" H 4750 3600 50  0001 C CNN
+F 4 "1%, " H 4750 3600 50  0001 C CNN "Characteristics"
 	1    4750 3600
 	1    0    0    -1
@@
 F 2 "Resistor_SMD:R_0805_2012Metric_Pad1.20x1.40mm_HandSolder" V 6830 3600 50  0001 C CNN
 F 3 "~" H 6900 3600 50  0001 C CNN
+F 4 "1%, min. 0.1 W" H 6900 3600 50  0001 C CNN "Characteristics"
 	1    6900 3600
 	1    0    0    -1
-$EndComp
-$Comp
-L Device:R_POT RV1
-U 1 1 61530ECD
-P 5100 4200
-F 0 "RV1" H 5030 4154 50  0000 R CNN
-F 1 "100 kΩ" H 5030 4245 50  0000 R CNN
-F 2 "mibe:Potentiometer_Bourns_3361P_Vertical" H 5100 4200 50  0001 C CNN
-F 3 "~" H 5100 4200 50  0001 C CNN
-	1    5100 4200
-	-1   0    0    1
 $EndComp
 $Comp
@@
 F 2 "Resistor_SMD:R_0805_2012Metric_Pad1.20x1.40mm_HandSolder" V 4430 4200 50  0001 C CNN
 F 3 "~" H 4500 4200 50  0001 C CNN
+F 4 "1%" H 4500 4200 50  0001 C CNN "Characteristics"
 	1    4500 4200
 	1    0    0    -1
@@
 Connection ~ 6300 4800
 Text Notes 8050 3100 0    50   ~ 0
-Imax: 401 mA due to R1
+Imax: 402 mA due to R1
 Text Notes 9450 3400 0    50   ~ 0
 Battery connected here
@@
 F 2 "Resistor_SMD:R_0805_2012Metric_Pad1.20x1.40mm_HandSolder" V 7730 3600 50  0001 C CNN
 F 3 "~" H 7800 3600 50  0001 C CNN
+F 4 "1%, min. 0.1 W" H 7800 3600 50  0001 C CNN "Characteristics"
 	1    7800 3600
 	1    0    0    -1
@@
 Wire Wire Line
 	4500 4050 4500 3900
+Text Label 4850 3350 0    50   ~ 0
+PROG
+Text Notes 5200 4400 0    50   ~ 0
+150 kΩ
 Text Notes 7950 4400 0    50   ~ 0
 Charging
 Text Notes 7050 4400 0    50   ~ 0
 Done
-Text Label 4850 3350 0    50   ~ 0
-PROG
+$Comp
+L Device:R_POT RV1
+U 1 1 61530ECD
+P 5100 4200
+F 0 "RV1" H 5030 4154 50  0000 R CNN
+F 1 "3361P-1-104G" H 5030 4245 50  0000 R CNN
+F 2 "mibe:Potentiometer_Bourns_3361P_Vertical" H 5100 4200 50  0001 C CNN
+F 3 "~" H 5100 4200 50  0001 C CNN
+F 4 "150 kΩ" H 5100 4200 50  0001 C CNN "Characteristics"
+	1    5100 4200
+	-1   0    0    1
+$EndComp
 $EndSCHEMATC
