File: MTG-life_counter/PCB/MTG-life_counter.sch (KiCad schematic (older format))
At the start: 39 parts, among them J2 AVR-ISP-6, Q1 IRLML6244, Q2 Si2301DS, Q3 Si2301DS, SW1 SW_Push, SW2 SW_Push, U2 AT90S4433-8P, U3 HDSP-H101, U4 HDSP-H101, Y1 8 MHz

Commit message: Add an on/off switch. This fixes #7.
Also fix ERC errors, rename nets to indicate the signals logic level, move some components a bit and update BOM & netlist.

This is rev. 22/2 of the board.
Parts:
- added SW3: SW_SPST, Connector_Wire:SolderWire-0.15sqmm_1x02_P4mm_D0.5mm_OD1.5mm, symbol Switch:SW_SPST
Connections:
- net +BATT: now also SW3.1 (A); no longer C6.1, D3.1 (K), L1.1, Q2.3 (D), Q3.3 (D), R17.1, R18.1, U2.7 (VCC)
- net SW_DEC renamed ~SW_DEC
- net SW_INC renamed ~SW_INC
- new net +3V8: C6.1, D3.1 (K), L1.1, Q2.3 (D), Q3.3 (D), R17.1, R18.1, SW3.2 (B), U2.7 (VCC)
Other:
- note added: "On / off switch"
Changed lines of the file:
@@
 	0    1    1    0
 $EndComp
-$Comp
-L power:GND #PWR06
-U 1 1 6141AFD6
-P 3500 4300
-F 0 "#PWR06" H 3500 4050 50  0001 C CNN
-F 1 "GND" H 3505 4127 50  0000 C CNN
-F 2 "" H 3500 4300 50  0001 C CNN
-F 3 "" H 3500 4300 50  0001 C CNN
-	1    3500 4300
-	1    0    0    -1
-$EndComp
-Wire Wire Line
-	3500 4300 3500 4250
-Wire Wire Line
-	3500 4250 3600 4250
 Wire Wire Line
 	3600 4250 3600 4150
-Connection ~ 3500 4250
 Wire Wire Line
 	3500 4250 3500 4150
@@
 $EndComp
 Wire Wire Line
-	4350 1150 5350 1150
-Wire Wire Line
 	5900 1150 5900 1200
 Connection ~ 4350 1150
@@
 Connection ~ 9150 6250
 Text Label 4300 1750 0    50   ~ 0
-SW_DEC
+~SW_DEC
 Text Label 4300 1850 0    50   ~ 0
-SW_INC
+~SW_INC
 Text Notes 8500 4150 0    50   ~ 0
 If: 15 mA\nVf: ~~ 1.73 V
@@
 	3600 1300 3600 1150
 $Comp
-L power:+BATT #PWR0101
-U 1 1 61C0CF65
-P 3050 1100
-F 0 "#PWR0101" H 3050 950 50  0001 C CNN
-F 1 "+BATT" H 3065 1273 50  0000 C CNN
-F 2 "" H 3050 1100 50  0001 C CNN
-F 3 "" H 3050 1100 50  0001 C CNN
-	1    3050 1100
-	1    0    0    -1
-$EndComp
-$Comp
-L power:+BATT #PWR0103
-U 1 1 61C18617
-P 9150 1500
-F 0 "#PWR0103" H 9150 1350 50  0001 C CNN
-F 1 "+BATT" H 9165 1673 50  0000 C CNN
-F 2 "" H 9150 1500 50  0001 C CNN
-F 3 "" H 9150 1500 50  0001 C CNN
-	1    9150 1500
-	1    0    0    -1
-$EndComp
-$Comp
-L power:+BATT #PWR05
-U 1 1 61C19A2C
-P 6200 5950
-F 0 "#PWR05" H 6200 5800 50  0001 C CNN
-F 1 "+BATT" H 6215 6123 50  0000 C CNN
-F 2 "" H 6200 5950 50  0001 C CNN
-F 3 "" H 6200 5950 50  0001 C CNN
-	1    6200 5950
-	1    0    0    -1
-$EndComp
-$Comp
 L Device:R R14
 U 1 1 61B08127
@@
 	0    -1   -1   0
 $EndComp
-NoConn ~ 4100 1650
 Wire Wire Line
 	8350 2100 8350 2250
@@
 Wire Wire Line
 	6200 6000 6200 5950
+NoConn ~ 4100 1650
+Wire Wire Line
+	3500 4250 3600 4250
+$Comp
+L power:GND #PWR06
+U 1 1 6141AFD6
+P 3500 4300
+F 0 "#PWR06" H 3500 4050 50  0001 C CNN
+F 1 "GND" H 3505 4127 50  0000 C CNN
+F 2 "" H 3500 4300 50  0001 C CNN
+F 3 "" H 3500 4300 50  0001 C CNN
+	1    3500 4300
+	1    0    0    -1
+$EndComp
+Connection ~ 3500 4250
+Wire Wire Line
+	3500 4300 3500 4250
+$Comp
+L power:+BATT #PWR010
+U 1 1 639A615B
+P 1250 4750
+F 0 "#PWR010" H 1250 4600 50  0001 C CNN
+F 1 "+BATT" H 1265 4923 50  0000 C CNN
+F 2 "" H 1250 4750 50  0001 C CNN
+F 3 "" H 1250 4750 50  0001 C CNN
+	1    1250 4750
+	1    0    0    -1
+$EndComp
+$Comp
+L power:+3V8 #PWR011
+U 1 1 639A6E0C
+P 1950 4750
+F 0 "#PWR011" H 1950 4600 50  0001 C CNN
+F 1 "+3V8" H 1965 4923 50  0000 C CNN
+F 2 "" H 1950 4750 50  0001 C CNN
+F 3 "" H 1950 4750 50  0001 C CNN
+	1    1950 4750
+	1    0    0    -1
+$EndComp
+Wire Wire Line
+	1250 4800 1400 4800
+Wire Wire Line
+	1800 4800 1950 4800
+$Comp
+L power:+3V8 #PWR0101
+U 1 1 639B609E
+P 9150 1500
+F 0 "#PWR0101" H 9150 1350 50  0001 C CNN
+F 1 "+3V8" H 9165 1673 50  0000 C CNN
+F 2 "" H 9150 1500 50  0001 C CNN
+F 3 "" H 9150 1500 50  0001 C CNN
+	1    9150 1500
+	1    0    0    -1
+$EndComp
+$Comp
+L power:+3V8 #PWR0102
+U 1 1 639B76CE
+P 3050 1100
+F 0 "#PWR0102" H 3050 950 50  0001 C CNN
+F 1 "+3V8" H 3065 1273 50  0000 C CNN
+F 2 "" H 3050 1100 50  0001 C CNN
+F 3 "" H 3050 1100 50  0001 C CNN
+	1    3050 1100
+	1    0    0    -1
+$EndComp
+Wire Wire Line
+	1250 4750 1250 4800
+Wire Wire Line
+	1950 4800 1950 4750
+Text Notes 1300 4950 0    50   ~ 0
+On / off switch
+Wire Wire Line
+	4350 1150 4850 1150
+$Comp
+L power:PWR_FLAG #FLG0104
+U 1 1 639CD435
+P 4850 1200
+F 0 "#FLG0104" H 4850 1275 50  0001 C CNN
+F 1 "PWR_FLAG" H 4850 1373 50  0000 C CNN
+F 2 "" H 4850 1200 50  0001 C CNN
+F 3 "~" H 4850 1200 50  0001 C CNN
+	1    4850 1200
+	-1   0    0    1
+$EndComp
+$Comp
+L power:PWR_FLAG #FLG0105
+U 1 1 639CDD80
+P 2000 4800
+F 0 "#FLG0105" H 2000 4875 50  0001 C CNN
+F 1 "PWR_FLAG" V 2000 4928 50  0000 L CNN
+F 2 "" H 2000 4800 50  0001 C CNN
+F 3 "~" H 2000 4800 50  0001 C CNN
+	1    2000 4800
+	0    1    1    0
+$EndComp
+Wire Wire Line
+	1950 4800 2000 4800
+Connection ~ 1950 4800
+Wire Wire Line
+	4850 1200 4850 1150
+Connection ~ 4850 1150
+Wire Wire Line
+	4850 1150 5350 1150
+$Comp
+L Switch:SW_SPST SW3
+U 1 1 639DD307
+P 1600 4800
+F 0 "SW3" H 1600 5035 50  0000 C CNN
+F 1 "SW_SPST" H 1600 4944 50  0000 C CNN
+F 2 "Connector_Wire:SolderWire-0.15sqmm_1x02_P4mm_D0.5mm_OD1.5mm" H 1600 4800 50  0001 C CNN
+F 3 "~" H 1600 4800 50  0001 C CNN
+	1    1600 4800
+	1    0    0    -1
+$EndComp
 Wire Bus Line
 	5250 3150 5250 4250
@@
 Wire Bus Line
 	9650 3150 9650 4250
+$Comp
+L power:+3V8 #PWR?
+U 1 1 639E8CE8
+P 6200 5950
+F 0 "#PWR?" H 6200 5800 50  0001 C CNN
+F 1 "+3V8" H 6215 6123 50  0000 C CNN
+F 2 "" H 6200 5950 50  0001 C CNN
+F 3 "" H 6200 5950 50  0001 C CNN
+	1    6200 5950
+	1    0    0    -1
+$EndComp
 $EndSCHEMATC
